File: ESC_4in1_G071_1S3_SIZ200.sch (KiCad schematic (older format))
At the start: 181 parts, among them J1 Conn_01x10, U1 STM32G071GBU6, U10 NCP81161MNTBG, U11 SIZ200DT-T1-GE3, U12 NCP81161MNTBG, U13 SIZ200DT-T1-GE3, U14 TPS630701, U15 TPS72733DSE, U16 INA186A2, U17 STM32G071GBU6, U18 NCP81161MNTBG, U19 SIZ200DT-T1-GE3, U2 NCP81161MNTBG, U20 NCP81161MNTBG, U21 STM32G071GBU6, U22 SIZ200DT-T1-GE3, U23 NCP81161MNTBG, U24 SIZ200DT-T1-GE3, U25 NCP81161MNTBG, U26 SIZ200DT-T1-GE3, U27 NCP81161MNTBG, U28 STM32G071GBU6, U29 SIZ200DT-T1-GE3, U3 SIZ200DT-T1-GE3, U30 NCP81161MNTBG, U31 SIZ200DT-T1-GE3, U4 NCP81161MNTBG, U5 SIZ200DT-T1-GE3, U6 NCP81161MNTBG, U7 SIZ200DT-T1-GE3, U8 NCP81161MNTBG, U9 SIZ200DT-T1-GE3

Commit message: update schematic and layout
Connections:
- net ESC1_A_DRVH: now also RN6.2 (R2.1); no longer RN4.1 (R1.1)
- net ESC1_A_DRVL: now also RN1.1 (R1.1); no longer RN3.2 (R2.1)
- net ESC1_A_GH: now also RN6.3 (R2.2); no longer RN4.4 (R1.2)
- net ESC1_A_GL: now also RN1.4 (R1.2); no longer RN3.3 (R2.2)
- net ESC1_B_DRVH: now also RN3.1 (R1.1); no longer RN1.2 (R2.1)
- net ESC1_B_GH: now also RN3.4 (R1.2); no longer RN1.3 (R2.2)
- net ESC1_C_DRVH: now also RN1.2 (R2.1); no longer RN3.1 (R1.1)
- net ESC1_C_GH: now also RN1.3 (R2.2); no longer RN3.4 (R1.2)
- net ESC2_C_DRVH: now also RN4.1 (R1.1); no longer RN6.2 (R2.1)
- net ESC2_C_DRVL: now also RN3.2 (R2.1); no longer RN1.1 (R1.1)
- net ESC2_C_GH: now also RN4.4 (R1.2); no longer RN6.3 (R2.2)
- net ESC2_C_GL: now also RN3.3 (R2.2); no longer RN1.4 (R1.2)
- net ESC3_A_DRVH: now also RN22.2 (R2.1); no longer R21.2
- net ESC3_A_DRVL: now also RN19.1 (R1.1); no longer RN19.2 (R2.1)
- net ESC3_A_GH: now also RN22.3 (R2.2); no longer R21.1
- net ESC3_A_GL: now also RN19.4 (R1.2); no longer RN19.3 (R2.2)
- net ESC3_B_DRVH: now also RN20.1 (R1.1); no longer R25.2
- net ESC3_B_DRVL: now also R25.2; no longer RN20.1 (R1.1)
- net ESC3_B_GH: now also RN20.4 (R1.2); no longer R25.1
- net ESC3_B_GL: now also R25.1; no longer RN20.4 (R1.2)
- net ESC3_C_DRVH: now also RN19.2 (R2.1); no longer RN19.1 (R1.1)
- net ESC3_C_DRVL: now also R21.2; no longer RN22.2 (R2.1)
- net ESC3_C_GH: now also RN19.3 (R2.2); no longer RN19.4 (R1.2)
- net ESC3_C_GL: now also R21.1; no longer RN22.3 (R2.2)
- net ESC4_A_DRVH: now also R24.2; no longer RN20.2 (R2.1)
- net ESC4_A_DRVL: now also RN14.2 (R2.1); no longer RN14.1 (R1.1)
- net ESC4_A_GH: now also R24.1; no longer RN20.3 (R2.2)
- net ESC4_A_GL: now also RN14.3 (R2.2); no longer RN14.4 (R1.2)
- net ESC4_B_DRVH: now also R20.2; no longer RN14.2 (R2.1)
- net ESC4_B_DRVL: now also RN22.1 (R1.1); no longer R24.2
- net ESC4_B_GH: now also R20.1; no longer RN14.3 (R2.2)
- net ESC4_B_GL: now also RN22.4 (R1.2); no longer R20.1
- net ESC4_C_DRVH: now also RN14.1 (R1.1); no longer RN22.1 (R1.1)
- net ESC4_C_DRVL: now also RN20.2 (R2.1); no longer R20.2
- net ESC4_C_GH: now also RN14.4 (R1.2); no longer RN22.4 (R1.2)
- net ESC4_C_GL: now also RN20.3 (R2.2); no longer R24.1
Changed lines of the file:
@@
 Connection ~ 24150 10900
 Connection ~ 13050 10900
+Text Label 11800 12300 0    50   ~ 0
+ESC4_B_DRVH
+Wire Wire Line
+	11800 12300 12350 12300
+Wire Wire Line
+	15950 12300 16500 12300
+Text Label 13100 12300 2    50   ~ 0
+ESC4_B_GH
+Text Label 17350 12300 2    50   ~ 0
+ESC4_B_GL
+Wire Wire Line
+	12650 12300 13100 12300
+Wire Wire Line
+	16900 12300 17350 12300
+Text Label 10150 12300 0    50   ~ 0
+ESC4_C_DRVH
+Text Label 19150 12400 0    50   ~ 0
+ESC4_C_DRVL
+Wire Wire Line
+	10150 12300 10700 12300
+Wire Wire Line
+	19150 12400 19700 12400
+Text Label 11550 12300 2    50   ~ 0
+ESC4_C_GH
+Text Label 20550 12400 2    50   ~ 0
+ESC4_C_GL
+Wire Wire Line
+	11100 12300 11550 12300
+Wire Wire Line
+	20100 12400 20550 12400
 Text Label 10150 12400 0    50   ~ 0
-ESC4_B_DRVH
+ESC4_A_DRVL
 Wire Wire Line
 	10150 12400 10700 12400
 Wire Wire Line
-	11800 12400 12350 12400
+	15950 12400 16500 12400
+Text Label 17350 12400 2    50   ~ 0
+ESC3_A_GH
 Text Label 11550 12400 2    50   ~ 0
-ESC4_B_GH
-Text Label 13100 12300 2    50   ~ 0
-ESC4_B_GL
+ESC4_A_GL
+Wire Wire Line
+	16900 12400 17350 12400
 Wire Wire Line
 	11100 12400 11550 12400
-Wire Wire Line
-	12650 12300 13100 12300
 Text Label 15950 12300 0    50   ~ 0
-ESC4_C_DRVH
-Text Label 11800 12300 0    50   ~ 0
-ESC4_C_DRVL
-Wire Wire Line
-	15950 12300 16500 12300
-Wire Wire Line
-	11800 12300 12350 12300
-Text Label 17350 12300 2    50   ~ 0
-ESC4_C_GH
-Text Label 13100 12400 2    50   ~ 0
-ESC4_C_GL
-Wire Wire Line
-	16900 12300 17350 12300
-Wire Wire Line
-	12650 12400 13100 12400
-Text Label 10150 12300 0    50   ~ 0
-ESC4_A_DRVL
-Wire Wire Line
-	10150 12300 10700 12300
-Wire Wire Line
-	13600 12300 14150 12300
-Text Label 14900 12300 2    50   ~ 0
-ESC3_A_GH
-Text Label 11550 12300 2    50   ~ 0
-ESC4_A_GL
-Wire Wire Line
-	14450 12300 14900 12300
-Wire Wire Line
-	11100 12300 11550 12300
-Text Label 11800 12400 0    50   ~ 0
 ESC4_B_DRVL
 $Comp
@@
 Text Label 17300 13950 2    50   ~ 0
 ESC3_A_DRVH
-Text Label 17350 12400 2    50   ~ 0
+Text Label 14900 12300 2    50   ~ 0
 ESC3_C_GL
 Wire Wire Line
-	16900 12400 17350 12400
+	14450 12300 14900 12300
+Text Label 13600 12300 0    50   ~ 0
+ESC3_C_DRVL
+Wire Wire Line
+	13600 12300 14150 12300
 Text Label 15950 12400 0    50   ~ 0
-ESC3_C_DRVL
-Wire Wire Line
-	15950 12400 16500 12400
-Text Label 13600 12300 0    50   ~ 0
 ESC3_A_DRVH
+Text Label 17600 12300 0    50   ~ 0
+ESC3_C_DRVH
+Wire Wire Line
+	17600 12300 18150 12300
 Text Label 17600 12400 0    50   ~ 0
-ESC3_C_DRVH
+ESC3_A_DRVL
 Wire Wire Line
 	17600 12400 18150 12400
-Text Label 17600 12300 0    50   ~ 0
-ESC3_A_DRVL
-Wire Wire Line
-	17600 12300 18150 12300
+Text Label 19000 12300 2    50   ~ 0
+ESC3_C_GH
+Wire Wire Line
+	18550 12300 19000 12300
 Text Label 19000 12400 2    50   ~ 0
-ESC3_C_GH
+ESC3_A_GL
 Wire Wire Line
 	18550 12400 19000 12400
-Text Label 19000 12300 2    50   ~ 0
-ESC3_A_GL
-Wire Wire Line
-	18550 12300 19000 12300
-Text Label 19150 12400 0    50   ~ 0
+Text Label 11800 12400 0    50   ~ 0
 ESC4_A_DRVH
 Wire Wire Line
-	19150 12400 19700 12400
+	11800 12400 12350 12400
+Text Label 13600 12400 0    50   ~ 0
+ESC3_B_DRVL
+Wire Wire Line
+	13600 12400 14150 12400
+Text Label 13100 12400 2    50   ~ 0
+ESC4_A_GH
+Wire Wire Line
+	12650 12400 13100 12400
+Text Label 14900 12400 2    50   ~ 0
+ESC3_B_GL
+Wire Wire Line
+	14450 12400 14900 12400
+Wire Wire Line
+	19150 12300 19700 12300
 Text Label 19150 12300 0    50   ~ 0
-ESC3_B_DRVL
-Wire Wire Line
-	19150 12300 19700 12300
-Text Label 20550 12400 2    50   ~ 0
-ESC4_A_GH
-Wire Wire Line
-	20100 12400 20550 12400
+ESC3_B_DRVH
 Text Label 20550 12300 2    50   ~ 0
-ESC3_B_GL
+ESC3_B_GH
 Wire Wire Line
 	20100 12300 20550 12300
-Wire Wire Line
-	13600 12400 14150 12400
-Text Label 13600 12400 0    50   ~ 0
-ESC3_B_DRVH
-Text Label 14900 12400 2    50   ~ 0
-ESC3_B_GH
-Wire Wire Line
-	14450 12400 14900 12400
 Text Label 28250 6150 2    50   ~ 0
 ESC2_A_DRVL
@@
 Text Label 28500 19050 0    50   ~ 0
 ESC1_C_GH
+Text Label 21750 12300 0    50   ~ 0
+ESC2_C_DRVH
+Wire Wire Line
+	21750 12300 22300 12300
+Text Label 23150 12300 2    50   ~ 0
+ESC2_C_GH
+Wire Wire Line
+	22700 12300 23150 12300
 Text Label 23350 12400 0    50   ~ 0
-ESC2_C_DRVH
+ESC1_A_DRVH
 Wire Wire Line
 	23350 12400 23900 12400
 Text Label 24750 12400 2    50   ~ 0
-ESC2_C_GH
+ESC1_A_GH
 Wire Wire Line
 	24300 12400 24750 12400
-Text Label 21750 12300 0    50   ~ 0
-ESC1_A_DRVH
-Wire Wire Line
-	21750 12300 22300 12300
-Text Label 23150 12300 2    50   ~ 0
-ESC1_A_GH
-Wire Wire Line
-	22700 12300 23150 12300
 Text Label 31500 12350 2    50   ~ 0
 ESC2_B_GH
@@
 	22700 12400 23150 12400
 Wire Wire Line
+	26550 12300 27100 12300
+Text Label 26550 12300 0    50   ~ 0
+ESC1_B_DRVH
+Text Label 27950 12300 2    50   ~ 0
+ESC1_B_GH
+Wire Wire Line
+	27500 12300 27950 12300
+Wire Wire Line
+	24950 12300 25500 12300
+Text Label 24950 12300 0    50   ~ 0
+ESC1_A_DRVL
+Text Label 26350 12300 2    50   ~ 0
+ESC1_A_GL
+Wire Wire Line
+	25900 12300 26350 12300
+Wire Wire Line
 	24950 12400 25500 12400
 Text Label 24950 12400 0    50   ~ 0
-ESC1_B_DRVH
+ESC1_C_DRVH
 Text Label 26350 12400 2    50   ~ 0
-ESC1_B_GH
+ESC1_C_GH
 Wire Wire Line
 	25900 12400 26350 12400
-Wire Wire Line
-	26550 12400 27100 12400
-Text Label 26550 12400 0    50   ~ 0
-ESC1_A_DRVL
-Text Label 27950 12400 2    50   ~ 0
-ESC1_A_GL
-Wire Wire Line
-	27500 12400 27950 12400
-Wire Wire Line
-	26550 12300 27100 12300
-Text Label 26550 12300 0    50   ~ 0
-ESC1_C_DRVH
-Text Label 27950 12300 2    50   ~ 0
-ESC1_C_GH
-Wire Wire Line
-	27500 12300 27950 12300
 $Comp
 L Connector:TestPoint TP15
@@
 Wire Wire Line
 	31050 12350 31500 12350
-Text Label 24950 12300 0    50   ~ 0
-ESC2_C_DRVL
-Wire Wire Line
-	24950 12300 25500 12300
-Text Label 26350 12300 2    50   ~ 0
+Text Label 27950 12400 2    50   ~ 0
 ESC2_C_GL
 Wire Wire Line
-	25900 12300 26350 12300
+	27500 12400 27950 12400
 Wire Wire Line
 	23400 11500 23950 11500
@@
 Text Notes 3500 3400 0    100  ~ 20
 Input: 1-3S (3...12.6 V)
+Wire Wire Line
+	26550 12400 27100 12400
+Text Label 26550 12400 0    50   ~ 0
+ESC2_C_DRVL
 $EndSCHEMATC

Commit message: update schematic and layout
Parts:
- removed R27, R28, R29, R30: 1k, Resistor_SMD:R_0402_1005Metric, symbol Device:R_Small
- removed RN2: 1k, 11_PSoC_FC_whoop:R_Array_Convex_4x0402_dense, symbol Device:R_Pack04
- added RN13, RN16, RN2, RN5: 1k, 11_PSoC_FC_whoop:R_Array_Convex_2x0402_dense, symbol Device:R_Pack02
Connections:
- net ESC1_IN: now also RN13.4 (R1.2)
- net ESC2_IN: now also RN13.3 (R2.2)
- net ESC3_IN: now also RN16.4 (R1.2)
- net ESC4_IN: now also RN16.3 (R2.2)
- net ESCx_tele: now also RN2.1 (R1.1), RN2.2 (R2.1), RN5.1 (R1.1), RN5.2 (R2.1)
- net ESC1_tele_o: now reaches U1.26 (PB6)
- net ESC1_tele_o: now also RN2.4 (R1.2)
- net at J1.8 (Pin_8): now also RN16.2 (R2.1)
- net at J1.7 (Pin_7): now also RN16.1 (R1.1)
- net at J1.6 (Pin_6): now also RN13.2 (R2.1)
- net at J1.5 (Pin_5): now also RN13.1 (R1.1)
- net ESC2_tele_o: now reaches U17.26 (PB6)
- net ESC2_tele_o: now also RN2.3 (R2.2)
- net ESC3_tele_o: now reaches U28.26 (PB6)
- net ESC3_tele_o: now also RN5.4 (R1.2)
- net ESC4_tele_o: now reaches U21.26 (PB6)
- net ESC4_tele_o: now also RN5.3 (R2.2)
Other:
- moved on the sheet: J1
