File: ESC_4in1_G071_1S3_SIZ200.sch (KiCad schematic (older format))
At the start: 180 parts, among them J1 Conn_01x10, U1 STM32G071GBU6, U10 NCP81161MNTBG, U11 SIZ200DT-T1-GE3, U12 NCP81161MNTBG, U13 SIZ200DT-T1-GE3, U14 TPS630701, U15 TPS72733DSE, U16 INA186A2, U17 STM32G071GBU6, U18 NCP81161MNTBG, U19 SIZ200DT-T1-GE3, U2 NCP81161MNTBG, U20 NCP81161MNTBG, U21 STM32G071GBU6, U22 SIZ200DT-T1-GE3, U23 NCP81161MNTBG, U24 SIZ200DT-T1-GE3, U25 NCP81161MNTBG, U26 SIZ200DT-T1-GE3, U27 NCP81161MNTBG, U28 STM32G071GBU6, U29 SIZ200DT-T1-GE3, U3 SIZ200DT-T1-GE3, U30 NCP81161MNTBG, U31 SIZ200DT-T1-GE3, U4 NCP81161MNTBG, U5 SIZ200DT-T1-GE3, U6 NCP81161MNTBG, U7 SIZ200DT-T1-GE3, U8 NCP81161MNTBG, U9 SIZ200DT-T1-GE3

Commit message: update schematic, layout and schematic pdf
Parts:
- C14: voltage (none) -> 25 V
- C16: type (none) -> T55A107M6R3C0045
- FB1, FB2: type (none) -> BLM18SG221TN1D
- J1: type (none) -> SM10B-SRSS-TB
- L1: value 1u -> 820 nH; type (none) -> DFE252012F-R82M=P2
Changed lines of the file:
@@
 P 10400 1000
 F 0 "L1" V 10219 1000 50  0000 C CNN
-F 1 "1u" V 10310 1000 50  0000 C CNN
+F 1 "820 nH" V 10310 1000 50  0000 C CNN
 F 2 "Inductor_SMD:L_Wuerth_MAPI-2510" H 10400 1000 50  0001 C CNN
 F 3 "~" H 10400 1000 50  0001 C CNN
+F 4 "DFE252012F-R82M=P2" V 10300 2100 50  0000 R CNN "type"
 	1    10400 1000
 	0    1    1    0
@@
 F 2 "11_PSoC_FC_whoop:C_0603_1608Metric_dense" H 9000 1800 50  0001 C CNN
 F 3 "~" H 9000 1800 50  0001 C CNN
+F 4 "25 V" H 8900 1950 50  0000 R CNN "voltage"
 	1    9000 1800
 	-1   0    0    1
@@
 F 2 "Capacitor_Tantalum_SMD:CP_EIA-3216-10_Kemet-I" H 11750 1800 50  0001 C CNN
 F 3 "~" H 11750 1800 50  0001 C CNN
+F 4 "T55A107M6R3C0045" H 12600 1650 50  0000 R CNN "type"
 	1    11750 1800
 	1    0    0    -1
@@
 F 2 "Inductor_SMD:L_0402_1005Metric" V 8230 1600 50  0001 C CNN
 F 3 "~" H 8300 1600 50  0001 C CNN
+F 4 "BLM18SG221TN1D" V 8400 1700 50  0000 R CNN "type"
 	1    8300 1600
 	0    1    1    0
@@
 F 2 "Inductor_SMD:L_0402_1005Metric" V 12080 1600 50  0001 C CNN
 F 3 "~" H 12150 1600 50  0001 C CNN
+F 4 "BLM18SG221TN1D" V 12250 2200 50  0000 R CNN "type"
 	1    12150 1600
 	0    1    1    0
@@
 F 2 "11_PSoC_FC_whoop:JST_SHL_SM10B-SHLS-TF_1x10-1MP_P1.00mm_Horizontal_dense" H 5300 7350 50  0001 C CNN
 F 3 "~" H 5300 7350 50  0001 C CNN
+F 4 "SM10B-SRSS-TB" H 6050 7150 50  0000 R CNN "type"
 	1    5300 7350
 	-1   0    0    -1

Commit message: cosmetic update
Parts:
- added C70: 10u, Capacitor_SMD:C_0402_1005Metric, symbol Device:C_Small
- C13: footprint 11_PSoC_FC_whoop:C_1206_3216Metric_dense -> 11_PSoC_FC_whoop:C_0805_2012Metric_dense; voltage (none) -> 25 V
Connections:
- net +3V3: now also C70.2
- net GND: now also C70.1
- net Batt-: now reaches R1.2, TP8.1, U16.5 (-)
Changed lines of the file:
@@
 Sheet 1 1
 Title "4in1 ESC, G071, 1-3S, SIZ200"
-Date "2021-02-03"
+Date "2021-02-25"
 Rev ""
 Comp "crteensy"
@@
 L power:+3V3 #PWR0104
 U 1 1 600F4EF0
-P 16650 1100
-F 0 "#PWR0104" H 16650 950 50  0001 C CNN
-F 1 "+3V3" H 16665 1273 50  0000 C CNN
-F 2 "" H 16650 1100 50  0001 C CNN
-F 3 "" H 16650 1100 50  0001 C CNN
-	1    16650 1100
+P 17050 1100
+F 0 "#PWR0104" H 17050 950 50  0001 C CNN
+F 1 "+3V3" H 17065 1273 50  0000 C CNN
+F 2 "" H 17050 1100 50  0001 C CNN
+F 3 "" H 17050 1100 50  0001 C CNN
+	1    17050 1100
 	1    0    0    -1
 $EndComp
@@
 F 0 "C13" H 8508 1754 50  0000 R CNN
 F 1 "10u" H 8508 1845 50  0000 R CNN
-F 2 "11_PSoC_FC_whoop:C_1206_3216Metric_dense" H 8600 1800 50  0001 C CNN
+F 2 "11_PSoC_FC_whoop:C_0805_2012Metric_dense" H 8600 1800 50  0001 C CNN
 F 3 "~" H 8600 1800 50  0001 C CNN
+F 4 "25 V" H 8600 1800 50  0001 C CNN "voltage"
 	1    8600 1800
 	-1   0    0    1
@@
 	16150 1200 16350 1200
 Wire Wire Line
-	16650 1200 16650 1100
+	17050 1200 17050 1100
 Wire Wire Line
 	14750 1100 14750 1200
@@
 Connection ~ 16350 1200
 Wire Wire Line
-	16350 1200 16650 1200
+	16350 1200 16800 1200
 $Comp
 L power:GND #PWR0149
@@
 	2150 700  2150 3100
 Wire Notes Line
-	14600 700  16950 700
+	14600 700  17250 700
 Wire Notes Line
-	16950 700  16950 2150
+	17250 700  17250 2150
 Wire Notes Line
-	16950 2150 14600 2150
+	17250 2150 14600 2150
 Wire Notes Line
 	14600 2150 14600 700
@@
 Text Label 7600 6350 2    50   ~ 0
 ESC1_tele_o
+$Comp
+L Device:C_Small C70
+U 1 1 608FFEA0
+P 16800 1450
+F 0 "C70" H 16708 1404 50  0000 R CNN
+F 1 "10u" H 16708 1495 50  0000 R CNN
+F 2 "Capacitor_SMD:C_0402_1005Metric" H 16800 1450 50  0001 C CNN
+F 3 "~" H 16800 1450 50  0001 C CNN
+	1    16800 1450
+	-1   0    0    1
+$EndComp
+Wire Wire Line
+	16800 1350 16800 1200
+$Comp
+L power:GND #PWR0287
+U 1 1 608FFEA7
+P 16800 1550
+F 0 "#PWR0287" H 16800 1300 50  0001 C CNN
+F 1 "GND" H 16805 1377 50  0000 C CNN
+F 2 "" H 16800 1550 50  0001 C CNN
+F 3 "" H 16800 1550 50  0001 C CNN
+	1    16800 1550
+	1    0    0    -1
+$EndComp
+Connection ~ 16800 1200
+Wire Wire Line
+	16800 1200 17050 1200
+Text Label 4200 5050 0    50   ~ 0
+Batt-
 $EndSCHEMATC

Commit message: update schematic, layout and doc
Parts:
- added D1: LED, LED_SMD:LED_0603_1608Metric, symbol Device:LED
- added R27: 1k, Resistor_SMD:R_0402_1005Metric, symbol Device:R
- added TP23, TP24: TestPoint, 11_PSoC_FC_whoop:TestPoint_Pad_D1.0mm_dense, symbol Connector:TestPoint
- U11, U13, U19, U22, U24, U26, U29, U3, U31, U5, U7, U9: footprint 11_PSoC_FC_whoop:PowerPAIR3.3x3.3 -> 11_PSoC_FC_whoop:PowerPAIR3.3x3.3_splitpaste
Connections:
- net +3V3: now also D1.2 (A), TP23.1
- net ESC1_A: now also RN8.2 (R2.1); no longer RN8.1 (R1.1)
- net ESC1_B: now also RN8.1 (R1.1); no longer RN8.2 (R2.1)
- net ESC1_MA: now also RN8.3 (R2.2); no longer RN8.4 (R1.2)
- net ESC1_MB: now also RN8.4 (R1.2); no longer RN8.3 (R2.2)
- net GND: now also R27.1, TP24.1
- new net: D1.1 (K), R27.2
Changed lines of the file:
@@
 Sheet 1 1
 Title "4in1 ESC, G071, 1-3S, SIZ200"
-Date "2021-02-25"
+Date "2021-02-28"
 Rev ""
 Comp "crteensy"
@@
 F 0 "U3" H 29300 14600 50  0000 L CNN
 F 1 "SIZ200DT-T1-GE3" H 29300 14500 50  0000 L CNN
-F 2 "11_PSoC_FC_whoop:PowerPAIR3.3x3.3" H 29850 14550 50  0001 C CNN
+F 2 "11_PSoC_FC_whoop:PowerPAIR3.3x3.3_splitpaste" H 29850 14550 50  0001 C CNN
 F 3 "" H 29850 14550 50  0001 C CNN
 	1    29250 14250
@@
 F 0 "U5" H 29300 17050 50  0000 L CNN
 F 1 "SIZ200DT-T1-GE3" H 29300 16950 50  0000 L CNN
-F 2 "11_PSoC_FC_whoop:PowerPAIR3.3x3.3" H 29850 17000 50  0001 C CNN
+F 2 "11_PSoC_FC_whoop:PowerPAIR3.3x3.3_splitpaste" H 29850 17000 50  0001 C CNN
 F 3 "" H 29850 17000 50  0001 C CNN
 	1    29250 16700
@@
 F 0 "U7" H 29300 19500 50  0000 L CNN
 F 1 "SIZ200DT-T1-GE3" H 29300 19400 50  0000 L CNN
-F 2 "11_PSoC_FC_whoop:PowerPAIR3.3x3.3" H 29850 19450 50  0001 C CNN
+F 2 "11_PSoC_FC_whoop:PowerPAIR3.3x3.3_splitpaste" H 29850 19450 50  0001 C CNN
 F 3 "" H 29850 19450 50  0001 C CNN
 	1    29250 19150
@@
 F 0 "U9" H 29300 6400 50  0000 L CNN
 F 1 "SIZ200DT-T1-GE3" H 29300 6300 50  0000 L CNN
-F 2 "11_PSoC_FC_whoop:PowerPAIR3.3x3.3" H 29850 6350 50  0001 C CNN
+F 2 "11_PSoC_FC_whoop:PowerPAIR3.3x3.3_splitpaste" H 29850 6350 50  0001 C CNN
 F 3 "" H 29850 6350 50  0001 C CNN
 	1    29250 6050
@@
 F 0 "U11" H 29300 8850 50  0000 L CNN
 F 1 "SIZ200DT-T1-GE3" H 29300 8750 50  0000 L CNN
-F 2 "11_PSoC_FC_whoop:PowerPAIR3.3x3.3" H 29850 8800 50  0001 C CNN
+F 2 "11_PSoC_FC_whoop:PowerPAIR3.3x3.3_splitpaste" H 29850 8800 50  0001 C CNN
 F 3 "" H 29850 8800 50  0001 C CNN
 	1    29250 8500
@@
 F 0 "U13" H 29300 11300 50  0000 L CNN
 F 1 "SIZ200DT-T1-GE3" H 29300 11200 50  0000 L CNN
-F 2 "11_PSoC_FC_whoop:PowerPAIR3.3x3.3" H 29850 11250 50  0001 C CNN
+F 2 "11_PSoC_FC_whoop:PowerPAIR3.3x3.3_splitpaste" H 29850 11250 50  0001 C CNN
 F 3 "" H 29850 11250 50  0001 C CNN
 	1    29250 10950
@@
 	2150 700  2150 3100
 Wire Notes Line
-	14600 700  17250 700
-Wire Notes Line
-	17250 700  17250 2150
-Wire Notes Line
-	17250 2150 14600 2150
-Wire Notes Line
-	14600 2150 14600 700
+	14600 2350 14600 700
 $Comp
 L power:GND #PWR0156
@@
 L Device:R_Pack02 RN8
 U 1 1 6020298A
-P 23950 18550
-F 0 "RN8" H 23770 18504 50  0000 R CNN
-F 1 "10k" H 23770 18595 50  0000 R CNN
-F 2 "11_PSoC_FC_whoop:R_Array_Convex_2x0402_dense" V 24225 18550 50  0001 C CNN
-F 3 "~" H 23950 18550 50  0001 C CNN
-	1    23950 18550
-	-1   0    0    1
+P 24050 18550
+F 0 "RN8" H 23870 18504 50  0000 R CNN
+F 1 "10k" H 23870 18595 50  0000 R CNN
+F 2 "11_PSoC_FC_whoop:R_Array_Convex_2x0402_dense" V 24325 18550 50  0001 C CNN
+F 3 "~" H 24050 18550 50  0001 C CNN
+	1    24050 18550
+	1    0    0    1
 $EndComp
 $Comp
@@
 F 0 "U26" H 18200 14600 50  0000 L CNN
 F 1 "SIZ200DT-T1-GE3" H 18200 14500 50  0000 L CNN
-F 2 "11_PSoC_FC_whoop:PowerPAIR3.3x3.3" H 18750 14550 50  0001 C CNN
+F 2 "11_PSoC_FC_whoop:PowerPAIR3.3x3.3_splitpaste" H 18750 14550 50  0001 C CNN
 F 3 "" H 18750 14550 50  0001 C CNN
 	1    18150 14250
@@
 F 0 "U29" H 18200 17050 50  0000 L CNN
 F 1 "SIZ200DT-T1-GE3" H 18200 16950 50  0000 L CNN
-F 2 "11_PSoC_FC_whoop:PowerPAIR3.3x3.3" H 18750 17000 50  0001 C CNN
+F 2 "11_PSoC_FC_whoop:PowerPAIR3.3x3.3_splitpaste" H 18750 17000 50  0001 C CNN
 F 3 "" H 18750 17000 50  0001 C CNN
 	1    18150 16700
@@
 F 0 "U31" H 18200 19500 50  0000 L CNN
 F 1 "SIZ200DT-T1-GE3" H 18200 19400 50  0000 L CNN
-F 2 "11_PSoC_FC_whoop:PowerPAIR3.3x3.3" H 18750 19450 50  0001 C CNN
+F 2 "11_PSoC_FC_whoop:PowerPAIR3.3x3.3_splitpaste" H 18750 19450 50  0001 C CNN
 F 3 "" H 18750 19450 50  0001 C CNN
 	1    18150 19150
@@
 F 0 "U22" H 18200 8850 50  0000 L CNN
 F 1 "SIZ200DT-T1-GE3" H 18200 8750 50  0000 L CNN
-F 2 "11_PSoC_FC_whoop:PowerPAIR3.3x3.3" H 18750 8800 50  0001 C CNN
+F 2 "11_PSoC_FC_whoop:PowerPAIR3.3x3.3_splitpaste" H 18750 8800 50  0001 C CNN
 F 3 "" H 18750 8800 50  0001 C CNN
 	1    18150 8500
@@
 F 0 "U24" H 18200 11300 50  0000 L CNN
 F 1 "SIZ200DT-T1-GE3" H 18200 11200 50  0000 L CNN
-F 2 "11_PSoC_FC_whoop:PowerPAIR3.3x3.3" H 18750 11250 50  0001 C CNN
+F 2 "11_PSoC_FC_whoop:PowerPAIR3.3x3.3_splitpaste" H 18750 11250 50  0001 C CNN
 F 3 "" H 18750 11250 50  0001 C CNN
 	1    18150 10950
@@
 F 0 "U19" H 18200 6400 50  0000 L CNN
 F 1 "SIZ200DT-T1-GE3" H 18200 6300 50  0000 L CNN
-F 2 "11_PSoC_FC_whoop:PowerPAIR3.3x3.3" H 18750 6350 50  0001 C CNN
+F 2 "11_PSoC_FC_whoop:PowerPAIR3.3x3.3_splitpaste" H 18750 6350 50  0001 C CNN
 F 3 "" H 18750 6350 50  0001 C CNN
 	1    18150 6050
@@
 Text Label 4200 5050 0    50   ~ 0
 Batt-
+Wire Notes Line
+	18250 2350 14600 2350
+Wire Notes Line
+	18250 700  18250 2350
+Wire Notes Line
+	14600 700  18250 700
+$Comp
+L Connector:TestPoint TP23
+U 1 1 6683BA44
+P 17900 1200
+F 0 "TP23" V 18095 1272 50  0000 C CNN
+F 1 "TestPoint" V 18004 1272 50  0000 C CNN
+F 2 "11_PSoC_FC_whoop:TestPoint_Pad_D1.0mm_dense" H 18100 1200 50  0001 C CNN
+F 3 "~" H 18100 1200 50  0001 C CNN
+	1    17900 1200
+	0    1    1    0
+$EndComp
+Wire Wire Line
+	17050 1200 17250 1200
+Connection ~ 17050 1200
+$Comp
+L Connector:TestPoint TP24
+U 1 1 668CE03A
+P 17900 1500
+F 0 "TP24" V 18095 1572 50  0000 C CNN
+F 1 "TestPoint" V 18004 1572 50  0000 C CNN
+F 2 "11_PSoC_FC_whoop:TestPoint_Pad_D1.0mm_dense" H 18100 1500 50  0001 C CNN
+F 3 "~" H 18100 1500 50  0001 C CNN
+	1    17900 1500
+	0    1    1    0
+$EndComp
+$Comp
+L power:GND #PWR0288
+U 1 1 668CE2AD
+P 17650 1550
+F 0 "#PWR0288" H 17650 1300 50  0001 C CNN
+F 1 "GND" H 17655 1377 50  0000 C CNN
+F 2 "" H 17650 1550 50  0001 C CNN
+F 3 "" H 17650 1550 50  0001 C CNN
+	1    17650 1550
+	1    0    0    -1
+$EndComp
+Wire Wire Line
+	17900 1500 17650 1500
+Wire Wire Line
+	17650 1500 17650 1550
+$Comp
+L Device:LED D1
+U 1 1 66D8485A
+P 17250 1450
+F 0 "D1" V 17289 1332 50  0000 R CNN
+F 1 "LED" V 17198 1332 50  0000 R CNN
+F 2 "LED_SMD:LED_0603_1608Metric" H 17250 1450 50  0001 C CNN
+F 3 "~" H 17250 1450 50  0001 C CNN
+	1    17250 1450
+	0    -1   -1   0
+$EndComp
+$Comp
+L Device:R R27
+U 1 1 66D8E6C9
+P 17250 1850
+F 0 "R27" V 17054 1850 50  0000 C CNN
+F 1 "1k" V 17145 1850 50  0000 C CNN
+F 2 "Resistor_SMD:R_0402_1005Metric" H 17250 1850 50  0001 C CNN
+F 3 "~" H 17250 1850 50  0001 C CNN
+	1    17250 1850
+	-1   0    0    1
+$EndComp
+$Comp
+L power:GND #PWR0289
+U 1 1 66D9C0DB
+P 17250 2050
+F 0 "#PWR0289" H 17250 1800 50  0001 C CNN
+F 1 "GND" H 17255 1877 50  0000 C CNN
+F 2 "" H 17250 2050 50  0001 C CNN
+F 3 "" H 17250 2050 50  0001 C CNN
+	1    17250 2050
+	1    0    0    -1
+$EndComp
+Wire Wire Line
+	17250 2050 17250 2000
+Wire Wire Line
+	17250 1700 17250 1600
+Wire Wire Line
+	17250 1200 17250 1300
+Connection ~ 17250 1200
+Wire Wire Line
+	17250 1200 17900 1200
 $EndSCHEMATC

Commit message: minor cosmetic updates
Parts:
- TP1, TP10, TP11, TP12, TP13, TP14, TP2, TP3, TP4, TP5, TP6, TP9: footprint 11_PSoC_FC_whoop:esc_pad -> 11_PSoC_FC_whoop:esc_pad_relaxed_n4
- TP7, TP8: footprint 11_PSoC_FC_whoop:batt_pad_wide -> 11_PSoC_FC_whoop:batt_pad_wide_relaxed
Changed lines of the file:
@@
 F 0 "TP1" H 30910 14344 50  0000 L CNN
 F 1 "TestPoint_Flag" H 30910 14253 50  0000 L CNN
-F 2 "11_PSoC_FC_whoop:esc_pad" H 30850 14250 50  0001 C CNN
+F 2 "11_PSoC_FC_whoop:esc_pad_relaxed_n4" H 30850 14250 50  0001 C CNN
 F 3 "~" H 30850 14250 50  0001 C CNN
 	1    30650 14250
@@
 F 0 "TP2" H 30910 16794 50  0000 L CNN
 F 1 "TestPoint_Flag" H 30910 16703 50  0000 L CNN
-F 2 "11_PSoC_FC_whoop:esc_pad" H 30850 16700 50  0001 C CNN
+F 2 "11_PSoC_FC_whoop:esc_pad_relaxed_n4" H 30850 16700 50  0001 C CNN
 F 3 "~" H 30850 16700 50  0001 C CNN
 	1    30650 16700
@@
 F 0 "TP3" H 30910 19244 50  0000 L CNN
 F 1 "TestPoint_Flag" H 30910 19153 50  0000 L CNN
-F 2 "11_PSoC_FC_whoop:esc_pad" H 30850 19150 50  0001 C CNN
+F 2 "11_PSoC_FC_whoop:esc_pad_relaxed_n4" H 30850 19150 50  0001 C CNN
 F 3 "~" H 30850 19150 50  0001 C CNN
 	1    30650 19150
@@
 F 0 "TP4" H 30910 6144 50  0000 L CNN
 F 1 "TestPoint_Flag" H 30910 6053 50  0000 L CNN
-F 2 "11_PSoC_FC_whoop:esc_pad" H 30850 6050 50  0001 C CNN
+F 2 "11_PSoC_FC_whoop:esc_pad_relaxed_n4" H 30850 6050 50  0001 C CNN
 F 3 "~" H 30850 6050 50  0001 C CNN
 	1    30650 6050
@@
 F 0 "TP5" H 30910 8594 50  0000 L CNN
 F 1 "TestPoint_Flag" H 30910 8503 50  0000 L CNN
-F 2 "11_PSoC_FC_whoop:esc_pad" H 30850 8500 50  0001 C CNN
+F 2 "11_PSoC_FC_whoop:esc_pad_relaxed_n4" H 30850 8500 50  0001 C CNN
 F 3 "~" H 30850 8500 50  0001 C CNN
 	1    30650 8500
@@
 F 0 "TP6" H 30910 11044 50  0000 L CNN
 F 1 "TestPoint_Flag" H 30910 10953 50  0000 L CNN
-F 2 "11_PSoC_FC_whoop:esc_pad" H 30850 10950 50  0001 C CNN
+F 2 "11_PSoC_FC_whoop:esc_pad_relaxed_n4" H 30850 10950 50  0001 C CNN
 F 3 "~" H 30850 10950 50  0001 C CNN
 	1    30650 10950
@@
 F 0 "TP8" H 3806 5052 50  0000 R CNN
 F 1 "TestPoint_Flag" H 3806 5143 50  0000 R CNN
-F 2 "11_PSoC_FC_whoop:batt_pad_wide" H 4050 5050 50  0001 C CNN
+F 2 "11_PSoC_FC_whoop:batt_pad_wide_relaxed" H 4050 5050 50  0001 C CNN
 F 3 "~" H 4050 5050 50  0001 C CNN
 	1    3850 5050
@@
 F 0 "TP7" H 3806 4144 50  0000 R CNN
 F 1 "TestPoint_Flag" H 3806 4053 50  0000 R CNN
-F 2 "11_PSoC_FC_whoop:batt_pad_wide" H 4050 4050 50  0001 C CNN
+F 2 "11_PSoC_FC_whoop:batt_pad_wide_relaxed" H 4050 4050 50  0001 C CNN
 F 3 "~" H 4050 4050 50  0001 C CNN
 	1    3850 4050
@@
 F 0 "TP12" H 19810 14344 50  0000 L CNN
 F 1 "TestPoint_Flag" H 19810 14253 50  0000 L CNN
-F 2 "11_PSoC_FC_whoop:esc_pad" H 19750 14250 50  0001 C CNN
+F 2 "11_PSoC_FC_whoop:esc_pad_relaxed_n4" H 19750 14250 50  0001 C CNN
 F 3 "~" H 19750 14250 50  0001 C CNN
 	1    19550 14250
@@
 F 0 "TP13" H 19810 16794 50  0000 L CNN
 F 1 "TestPoint_Flag" H 19810 16703 50  0000 L CNN
-F 2 "11_PSoC_FC_whoop:esc_pad" H 19750 16700 50  0001 C CNN
+F 2 "11_PSoC_FC_whoop:esc_pad_relaxed_n4" H 19750 16700 50  0001 C CNN
 F 3 "~" H 19750 16700 50  0001 C CNN
 	1    19550 16700
@@
 F 0 "TP14" H 19810 19244 50  0000 L CNN
 F 1 "TestPoint_Flag" H 19810 19153 50  0000 L CNN
-F 2 "11_PSoC_FC_whoop:esc_pad" H 19750 19150 50  0001 C CNN
+F 2 "11_PSoC_FC_whoop:esc_pad_relaxed_n4" H 19750 19150 50  0001 C CNN
 F 3 "~" H 19750 19150 50  0001 C CNN
 	1    19550 19150
@@
 F 0 "TP9" H 19810 6144 50  0000 L CNN
 F 1 "TestPoint_Flag" H 19810 6053 50  0000 L CNN
-F 2 "11_PSoC_FC_whoop:esc_pad" H 19750 6050 50  0001 C CNN
+F 2 "11_PSoC_FC_whoop:esc_pad_relaxed_n4" H 19750 6050 50  0001 C CNN
 F 3 "~" H 19750 6050 50  0001 C CNN
 	1    19550 6050
@@
 F 0 "TP10" H 19810 8594 50  0000 L CNN
 F 1 "TestPoint_Flag" H 19810 8503 50  0000 L CNN
-F 2 "11_PSoC_FC_whoop:esc_pad" H 19750 8500 50  0001 C CNN
+F 2 "11_PSoC_FC_whoop:esc_pad_relaxed_n4" H 19750 8500 50  0001 C CNN
 F 3 "~" H 19750 8500 50  0001 C CNN
 	1    19550 8500
@@
 F 0 "TP11" H 19810 11044 50  0000 L CNN
 F 1 "TestPoint_Flag" H 19810 10953 50  0000 L CNN
-F 2 "11_PSoC_FC_whoop:esc_pad" H 19750 10950 50  0001 C CNN
+F 2 "11_PSoC_FC_whoop:esc_pad_relaxed_n4" H 19750 10950 50  0001 C CNN
 F 3 "~" H 19750 10950 50  0001 C CNN
 	1    19550 10950
