File: ESC_4in1_G071_1S3_SIZ200.kicad_pcb (KiCad board)
At the start: 4 copper layers, 28 x 28 mm, 185 parts, among them J1 Conn_01x10, U1 STM32G071GBU6, U10 NCP81161MNTBG, U11 SIZ200DT-T1-GE3, U12 NCP81161MNTBG, U13 SIZ200DT-T1-GE3, U14 TPS630701, U15 TPS72733DSE, U16 INA186A2, U17 STM32G071GBU6, U18 NCP81161MNTBG, U19 SIZ200DT-T1-GE3, U2 NCP81161MNTBG, U20 NCP81161MNTBG, U21 STM32G071GBU6, U22 SIZ200DT-T1-GE3, U23 NCP81161MNTBG, U24 SIZ200DT-T1-GE3, U25 NCP81161MNTBG, U26 SIZ200DT-T1-GE3, U27 NCP81161MNTBG, U28 STM32G071GBU6, U29 SIZ200DT-T1-GE3, U3 SIZ200DT-T1-GE3, U30 NCP81161MNTBG, U31 SIZ200DT-T1-GE3, U4 NCP81161MNTBG, U5 SIZ200DT-T1-GE3, U6 NCP81161MNTBG, U7 SIZ200DT-T1-GE3, U8 NCP81161MNTBG, U9 SIZ200DT-T1-GE3

Commit message: minor cosmetic updates
Parts:
- TP1, TP10, TP11, TP12, TP13, TP14, TP2, TP3, TP4, TP5, TP6, TP9: footprint 11_PSoC_FC_whoop:esc_pad -> 11_PSoC_FC_whoop:esc_pad_relaxed_n4
- TP7, TP8: footprint 11_PSoC_FC_whoop:batt_pad_wide -> 11_PSoC_FC_whoop:batt_pad_wide_relaxed
- moved TP8 0.50 mm to (139.5, 89.0)
- moved R1 0.18 mm to (140.9, 86.1)
- moved C37 0.10 mm to (131.0, 86.0)
Routing:
- net /Batt-: track 6.89 -> 3.03 mm
- net GND: track 144.0 -> 143.0 mm, vias 87 -> 89
- net +BATT: track 86.1 -> 86.8 mm
