File: ESC_4in1_G071_1S3_SIZ200_badDCDC.kicad_pcb (KiCad board)
At the start: 4 copper layers, 28 x 28 mm, 185 parts, among them J1 Conn_01x10, U1 STM32G071GBU6, U10 NCP81161MNTBG, U11 SIZ200DT-T1-GE3, U12 NCP81161MNTBG, U13 SIZ200DT-T1-GE3, U14 TPS630701, U15 TPS72733DSE, U16 INA186A2, U17 STM32G071GBU6, U18 NCP81161MNTBG, U19 SIZ200DT-T1-GE3, U2 NCP81161MNTBG, U20 NCP81161MNTBG, U21 STM32G071GBU6, U22 SIZ200DT-T1-GE3, U23 NCP81161MNTBG, U24 SIZ200DT-T1-GE3, U25 NCP81161MNTBG, U26 SIZ200DT-T1-GE3, U27 NCP81161MNTBG, U28 STM32G071GBU6, U29 SIZ200DT-T1-GE3, U3 SIZ200DT-T1-GE3, U30 NCP81161MNTBG, U31 SIZ200DT-T1-GE3, U4 NCP81161MNTBG, U5 SIZ200DT-T1-GE3, U6 NCP81161MNTBG, U7 SIZ200DT-T1-GE3, U8 NCP81161MNTBG, U9 SIZ200DT-T1-GE3

Commit message: update DCDC layout
Parts:
- moved FB1 7.17 mm to (137.5, 62.0), turned to 0 degrees
- moved C17 4.20 mm to (140.4, 63.8), turned to 270 degrees
- moved L1 3.47 mm to (133.7, 64.4), turned to 90 degrees
- moved C15 3.38 mm to (135.9, 65.9)
- moved C14 2.52 mm to (135.9, 62.9), turned to 90 degrees
- moved U14 2.27 mm to (138.2, 64.4), turned to 270 degrees
- moved C16 1.77 mm to (142.0, 63.8)
- moved C13 1.32 mm to (131.2, 64.4), turned to 90 degrees
- moved FB2 0.46 mm to (140.4, 65.8), turned to 90 degrees
- moved R2 0.09 mm to (138.7, 67.2)
- moved RN10 0.07 mm to (138.6, 69.1)
Routing:
- net GND: track 125.2 -> 141.0 mm, vias 94 -> 86
- net Net-(C13-Pad2): track 2.52 -> 9.50 mm, vias 2 -> 0
- net Net-(C15-Pad2): track 2.06 -> 7.52 mm, vias 2 -> 0
- net Net-(L1-Pad2): track 2.57 -> 4.68 mm
- net +BATT: track 88.6 -> 87.1 mm, vias 52 -> 54
- net Net-(L1-Pad1): track 2.57 -> 4.05 mm
- net +5V: track 41.6 -> 42.5 mm, vias 15 -> 16
- removed copper zone on B.Cu, net Net-(C13-Pad2)
