File: backup_20210413_badVias/ESC_4in1_G071_1S3_SIZ200.sch (KiCad schematic (older format))
At the start: 191 parts, among them J1 Conn_01x10, U1 STM32G071GBU6, U10 NCP81161MNTBG, U11 SIZ200DT-T1-GE3, U12 NCP81161MNTBG, U13 SIZ200DT-T1-GE3, U14 TPS630701, U15 TPS72733DSE, U16 INA186A2, U17 STM32G071GBU6, U18 NCP81161MNTBG, U19 SIZ200DT-T1-GE3, U2 NCP81161MNTBG, U20 NCP81161MNTBG, U21 STM32G071GBU6, U22 SIZ200DT-T1-GE3, U23 NCP81161MNTBG, U24 SIZ200DT-T1-GE3, U25 NCP81161MNTBG, U26 SIZ200DT-T1-GE3, U27 NCP81161MNTBG, U28 STM32G071GBU6, U29 SIZ200DT-T1-GE3, U3 SIZ200DT-T1-GE3, U30 NCP81161MNTBG, U31 SIZ200DT-T1-GE3, U4 NCP81161MNTBG, U5 SIZ200DT-T1-GE3, U6 NCP81161MNTBG, U7 SIZ200DT-T1-GE3, U8 NCP81161MNTBG, U9 SIZ200DT-T1-GE3

Commit message: general redesign 1 current sensor per ESC
Parts:
- removed R28, R29, R30, R31, R32, R33, R34, R35, R38, R39, R40, R41, R42, R43, R44, R45: 10R0, Resistor_SMD:R_0402_1005Metric, symbol Device:R
- removed R36, R37: 10k, Resistor_SMD:R_0402_1005Metric, symbol Device:R_Small
- added C57, C58, C59, C60, C61, C62, C64, C65, C66, C67, C68, C69: 10u, Capacitor_SMD:C_0402_1005Metric, symbol Device:C_Small
- C11, C23, C26, C28, C30, C33, C35, C4, C5, C6, C7, C9: value 1u -> 100n
- R1: footprint 11_PSoC_FC_whoop:C_0603_1608Metric_dense -> Resistor_SMD:R_1206_3216Metric
- TP1, TP10, TP11, TP12, TP13, TP14, TP2, TP3, TP4, TP5, TP6, TP9: footprint 11_PSoC_FC_whoop:ESC_Pad_2.0x2.0mm -> 11_PSoC_FC_whoop:esc_pad_relaxed_n4
Connections:
- net +3V3: now also U16.3 (V+)
- net +5V: now also C57.2, C58.2, C59.2, C60.2, C61.2, C62.2, C64.2, C65.2, C66.2, C67.2, C68.2, C69.2; no longer U16.3 (V+)
- net +BATT: now also C37.2, C38.2, C39.2, U19.2 (D1), U22.2 (D1), U24.2 (D1); no longer R1.1, U16.4 (+)
- net ESC1_A_DRVH: now also RN6.2 (R2.1)
- net ESC1_A_DRVL: now also RN1.1 (R1.1)
- net ESC1_A_GH: now also RN6.3 (R2.2)
- net ESC1_A_GL: now also RN1.4 (R1.2)
- net ESC1_B_DRVH: now also RN3.1 (R1.1)
- net ESC1_B_GH: now also RN3.4 (R1.2)
- net ESC1_C_DRVH: now also RN1.2 (R2.1)
- net ESC1_C_GH: now also RN1.3 (R2.2)
- net ESC2_A: now also RN10.1 (R1.1)
- net ESC2_A_DRVL: now also RN4.2 (R2.1)
- net ESC2_A_GL: now also RN4.3 (R2.2)
- net ESC2_B: now also RN10.2 (R2.1)
- net ESC2_B_DRVL: now also RN6.1 (R1.1)
- net ESC2_B_GL: now also RN6.4 (R1.2)
- net ESC2_C_DRVH: now also RN4.1 (R1.1)
- net ESC2_C_DRVL: now also RN3.2 (R2.1)
- net ESC2_C_GH: now also RN4.4 (R1.2)
- net ESC2_C_GL: now also RN3.3 (R2.2)
- net ESC2_MA: now also RN10.4 (R1.2)
- net ESC2_MB: now also RN10.3 (R2.2)
- net ESC3_A_DRVH: now also RN22.2 (R2.1)
- net ESC3_A_DRVL: now also RN19.1 (R1.1)
- net ESC3_A_GH: now also RN22.3 (R2.2)
- net ESC3_A_GL: now also RN19.4 (R1.2)
- net ESC3_B_DRVH: now also RN20.1 (R1.1)
- net ESC3_B_GH: now also RN20.4 (R1.2)
- net ESC3_C_DRVH: now also RN19.2 (R2.1)
- net ESC3_C_GH: now also RN19.3 (R2.2)
- net ESC4_A_DRVL: now also RN14.2 (R2.1)
- net ESC4_A_GL: now also RN14.3 (R2.2)
- net ESC4_B_DRVL: now also RN22.1 (R1.1)
- net ESC4_B_GL: now also RN22.4 (R1.2)
- net ESC4_C_DRVH: now also RN14.1 (R1.1)
- net ESC4_C_DRVL: now also RN20.2 (R2.1)
- net ESC4_C_GH: now also RN14.4 (R1.2)
- net ESC4_C_GL: now also RN20.3 (R2.2)
- net GND: now also R1.1, U16.4 (+), C57.1, C58.1, C59.1, C60.1, C61.1, C62.1, C64.1, C65.1, C66.1, C67.1, C68.1, C69.1; no longer TP8.1
- removed net VESC4: C37.2, C38.2, C39.2, R1.2, U16.5 (-), U19.2 (D1), U22.2 (D1), U24.2 (D1)
- new net Batt-: R1.2, TP8.1, U16.5 (-)
Other:
- note removed: "assign MCU current input pin!"
- moved on the sheet: C20, C25, C37, C38, C39, C63, R1, R2, RN1, RN10, RN14, RN19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
